File: ATMega Dev Board.kicad_sch (KiCad schematic)
At the start: 40 parts, among them J1 Conn_01x09, J2 Conn_01x04, J3 Conn_01x09, J4 SPI header, J5 USB-C_31-M-12, Q1 S8050, SW1 SW_SPST, SW2 SW_SPST, U1 ATmega32A-A, U2 CH340C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

Commit message: Improved VCC routing
Parts:
- J5: footprint Connector_USB:USB_C_Receptacle_HRO_TYPE-C-31-M-12 -> FTBLib:USB_C_Receptacle_HRO_TYPE-C-31-M-12
Changed lines of the file:
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@@
 			)
 		)
-		(property "Footprint" "Connector_USB:USB_C_Receptacle_HRO_TYPE-C-31-M-12"
+		(property "Footprint" "FTBLib:USB_C_Receptacle_HRO_TYPE-C-31-M-12"
 			(at 210.82 49.53 0)
 			(effects

Commit message: Better traces
Parts:
- removed C6: 0.1u, Capacitor_SMD:C_0603_1608Metric, symbol Device:C_Small
- R1: value 4k7 -> 10k; LCSC C23162 -> C25804
Changed lines of the file:
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@@
-	(symbol
-		(lib_id "Device:C_Small")
-		(at 50.8 39.37 0)
-		(unit 1)
-		(exclude_from_sim no)
-		(in_bom yes)
-		(on_board yes)
-		(dnp no)
-		(property "Reference" "C6"
-			(at 44.704 38.1 0)
-			(effects
-				(font
-					(size 1.27 1.27)
-				)
-				(justify left)
-			)
-		)
-		(property "Value" "0.1u"
-			(at 44.45 40.132 0)
-			(effects
-				(font
-					(size 1.27 1.27)
-				)
-				(justify left)
-			)
-		)
-		(property "Footprint" "Capacitor_SMD:C_0603_1608Metric"
-			(at 50.8 39.37 0)
-			(effects
-				(font
-					(size 1.27 1.27)
-				)
-				(hide yes)
-			)
-		)
-		(property "Datasheet" "~"
-			(at 50.8 39.37 0)
-			(effects
-				(font
-					(size 1.27 1.27)
-				)
-				(hide yes)
-			)
-		)
-		(property "Description" "Unpolarized capacitor, small symbol"
-			(at 50.8 39.37 0)
-			(effects
-				(font
-					(size 1.27 1.27)
-				)
-				(hide yes)
-			)
-		)
-		(property "LCSC" "C14663"
-			(at 44.704 38.1 0)
-			(effects
-				(font
-					(size 1.27 1.27)
-				)
-				(hide yes)
-			)
-		)
-		(pin "2"
-		)
-		(pin "1"
-		)
-		(instances
-			(project "FTBTimer"
-				(path "/4c984bef-51cd-42e2-a43e-17b5e9351018"
-					(reference "C3")
-					(unit 1)
-				)
-			)
-			(project ""
-				(path "/70bbf962-aa97-42ae-8e7e-b12a946a1ea0"
-					(reference "C6")
-					(unit 1)
-				)
-			)
-		)
-	)
 	(symbol
 		(lib_id "Device:C_Small")
@@
 	(symbol
 		(lib_id "power:GND")
-		(at 50.8 41.91 0)
-		(unit 1)
-		(exclude_from_sim no)
-		(in_bom yes)
-		(on_board yes)
-		(dnp no)
-		(property "Reference" "#PWR03"
-			(at 50.8 48.26 0)
-			(effects
-				(font
-					(size 1.27 1.27)
-				)
-				(hide yes)
-			)
-		)
-		(property "Value" "GND"
-			(at 46.99 43.688 0)
-			(effects
-				(font
-					(size 1.27 1.27)
-				)
-			)
-		)
-		(property "Footprint" ""
-			(at 50.8 41.91 0)
-			(effects
-				(font
-					(size 1.27 1.27)
-				)
-				(hide yes)
-			)
-		)
-		(property "Datasheet" ""
-			(at 50.8 41.91 0)
-			(effects
-				(font
-					(size 1.27 1.27)
-				)
-				(hide yes)
-			)
-		)
-		(property "Description" "Power symbol creates a global label with name \"GND\" , ground"
-			(at 50.8 41.91 0)
-			(effects
-				(font
-					(size 1.27 1.27)
-				)
-				(hide yes)
-			)
-		)
-		(pin "1"
-		)
-		(instances
-			(project "ATMega Dev Board"
-				(path "/70bbf962-aa97-42ae-8e7e-b12a946a1ea0"
-					(reference "#PWR03")
-					(unit 1)
-				)
-			)
-		)
-	)
-	(symbol
-		(lib_id "power:GND")
 		(at 194.31 31.75 0)
 		(unit 1)
@@
 			)
 		)
-		(property "Value" "4k7"
-			(at 51.816 35.052 0)
+		(property "Value" "10k"
+			(at 50.8 36.068 90)
 			(effects
 				(font
@@
 			)
 		)
-		(property "LCSC" "C23162"
+		(property "LCSC" "C25804"
 			(at 50.8 34.29 0)
 			(effects
